File: Flame60/pcb/PCB_Layer1/Flame60_PCB_Layer1.kicad_pcb (KiCad board)
At the start: 2 copper layers, 298 x 108 mm, 137 parts, among them J1 Conn_01x04, J2 Conn_01x04, J3 Conn_01x04, J4 Conn_01x02, J5 Conn_01x02, SW1 SW_Esc, SW10 SW_W, SW11 SW_S, SW12 SW_X, SW13 SW_3, SW14 SW_E, SW15 SW_D, SW16 SW_C, SW17 SW_4, SW18 SW_R, SW19 SW_F, SW2 SW_Tab, SW20 SW_V, SW21 SW_5, SW22 SW_T, SW23 SW_G, SW24 SW_B, SW25 SW_6, SW26 SW_Y, SW27 SW_H, SW28 SW_N, SW29 SW_7, SW3 SW_Control, SW30 SW_U, SW31 SW_J, SW32 SW_M, SW33 SW_8, SW34 SW_I, SW35 SW_K, SW36 SW_<, SW37 SW_9, SW38 SW_O, SW39 SW_L, SW4 SW_Shift(L), SW40 SW_>, SW41 SW_0, SW42 SW_P, SW43 SW_;, SW44 SW_/, SW45 SW_-, SW46 SW_[, SW47 SW_', SW48 SW_Shift(R), SW49 SW_=, SW5 SW_1, SW50 SW_], SW51 SW_Return, SW52 SW_Fn, SW53 SW_\, SW54 SW_◇(L), SW55 SW_◇(R), SW56 SW_Delete, SW57 SW_Space, SW58 SW_`, SW59 SW_Alt(L), SW6 SW_Q, SW60 SW_Alt(R), SW7 SW_A, SW8 SW_Z, SW9 SW_2

Commit message: fix: remove redundant wires
Routing:
- net Net-(D11-Pad2): track 16.1 -> 9.15 mm
- net Net-(D35-Pad2): track 16.1 -> 9.15 mm
Changed lines of the file:
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@@
   (segment (start 140.49375 108.875) (end 140.49375 106.84) (width 0.25) (layer "F.Cu") (net 14))
   (segment (start 140.17625 106.83875) (end 140.49375 107.15625) (width 0.25) (layer "F.Cu") (net 14))
-  (segment (start 133.50875 106.83875) (end 140.4925 106.83875) (width 0.25) (layer "B.Cu") (net 14))
   (segment (start 140.4925 106.83875) (end 140.49375 106.84) (width 0.25) (layer "B.Cu") (net 14))
   (segment (start 150.0175 125.88875) (end 150.01875 125.89) (width 0.25) (layer "F.Cu") (net 15))
@@
   (segment (start 254.79375 108.875) (end 254.79375 106.84) (width 0.25) (layer "F.Cu") (net 48))
   (segment (start 254.7925 106.83875) (end 254.79375 106.84) (width 0.25) (layer "B.Cu") (net 48))
-  (segment (start 247.80875 106.83875) (end 254.7925 106.83875) (width 0.25) (layer "B.Cu") (net 48))
   (segment (start 264.3175 125.88875) (end 264.31875 125.89) (width 0.25) (layer "F.Cu") (net 49))
   (segment (start 264.31875 125.89) (end 264.31875 127.925) (width 0.25) (layer "F.Cu") (net 49))

Commit message: feat: consistency of wiring
Routing:
- net Row6: track 313.6 -> 318.4 mm
- net Row4: track 285.0 -> 286.0 mm
- net Col7: track 374.1 -> 374.8 mm
Other:
- board text added: "Flame60 ver1.1 @PCB L1 Designed by multifeb13"
- board text removed: "Flame60 ver1.0 @PCB L1 Designed by multifeb13"
