File: Flame60/pcb/PCB_Layer2/Flame60_PCB_Layer2.kicad_pcb (KiCad board)
At the start: 2 copper layers, 298 x 108 mm, 20 parts, among them J1 Conn_01x04, J2 Conn_01x04, J3 Conn_01x04, J4 Conn_01x02, J5 Conn_01x02, SW1 SW_PUSH, U1 ProMicro

Commit message: feat: consistency of wiring
Other:
- board text added: "Flame60 ver1.1 @PCB L2 Designed by multifeb13"
- board text removed: "Flame60 ver1.0 @PCB L2 Designed by multifeb13"
Changed lines of the file:
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@@
   (gr_line (start 359 58) (end 65 58) (layer "Edge.Cuts") (width 0.1))
   (gr_arc (start 65 166) (mid 63.585786 165.414214) (end 63 164) (layer "Edge.Cuts") (width 0.1))
-  (gr_text "Flame60 ver1.0 @PCB L2 Designed by multifeb13" (at 353 163) (layer "F.SilkS")
+  (gr_text "Flame60 ver1.1 @PCB L2 Designed by multifeb13" (at 353 163) (layer "F.SilkS")
     (effects (font (size 1 1) (thickness 0.125)) (justify right))
   )
@@
   (segment (start 90.01125 84.135001) (end 71.4 102.746251) (width 0.25) (layer "F.Cu") (net 14))
   (segment (start 71.4 102.746251) (end 71.4 125) (width 0.25) (layer "F.Cu") (net 14))
-  (segment (start 71.4 127.54) (end 72.575 126.365) (width 0.25) (layer "F.Cu") (net 15))
-  (segment (start 72.575 104.111251) (end 90.01125 86.675001) (width 0.25) (layer "F.Cu") (net 15))
-  (segment (start 72.575 126.365) (end 72.575 104.111251) (width 0.25) (layer "F.Cu") (net 15))
-  (segment (start 90.01125 89.215001) (end 74 105.226251) (width 0.25) (layer "F.Cu") (net 16))
-  (segment (start 74 127.48) (end 71.4 130.08) (width 0.25) (layer "F.Cu") (net 16))
-  (segment (start 74 105.226251) (end 74 127.48) (width 0.25) (layer "F.Cu") (net 16))
-  (segment (start 71.4 132.62) (end 75.5 128.52) (width 0.25) (layer "F.Cu") (net 17))
-  (segment (start 75.5 107) (end 90.01125 92.48875) (width 0.25) (layer "F.Cu") (net 17))
-  (segment (start 90.01125 92.48875) (end 90.01125 91.755001) (width 0.25) (layer "F.Cu") (net 17))
-  (segment (start 75.5 128.52) (end 75.5 107) (width 0.25) (layer "F.Cu") (net 17))
+  (segment (start 73 125.94) (end 73 103.686251) (width 0.25) (layer "F.Cu") (net 15))
+  (segment (start 73 103.686251) (end 90.01125 86.675001) (width 0.25) (layer "F.Cu") (net 15))
+  (segment (start 71.4 127.54) (end 73 125.94) (width 0.25) (layer "F.Cu") (net 15))
+  (segment (start 74.5 104.726251) (end 74.5 126.98) (width 0.25) (layer "F.Cu") (net 16))
+  (segment (start 74.5 126.98) (end 71.4 130.08) (width 0.25) (layer "F.Cu") (net 16))
+  (segment (start 90.01125 89.215001) (end 74.5 104.726251) (width 0.25) (layer "F.Cu") (net 16))
+  (segment (start 76 128.02) (end 76 105.5) (width 0.25) (layer "F.Cu") (net 17))
+  (segment (start 71.4 132.62) (end 76 128.02) (width 0.25) (layer "F.Cu") (net 17))
+  (segment (start 76 105.5) (end 89.744999 91.755001) (width 0.25) (layer "F.Cu") (net 17))
+  (segment (start 89.744999 91.755001) (end 90.01125 91.755001) (width 0.25) (layer "F.Cu") (net 17))
   (segment (start 284.803749 73.975001) (end 292.735 66.04375) (width 0.25) (layer "F.Cu") (net 18))
   (segment (start 105.25125 73.975001) (end 284.803749 73.975001) (width 0.25) (layer "F.Cu") (net 18))
