File: Water47/pcb/PCB_Layer/Water47_PCB_Layer.kicad_pcb (KiCad board)
At the start: 2 copper layers, 260 x 77.5 mm, 107 parts, among them SW1 Esc, SW10 O, SW11 P, SW12 -, SW13 Del, SW14 Cmd, SW15 A, SW16 S, SW17 D, SW18 F, SW19 G, SW2 Q, SW20 H, SW21 J, SW22 K, SW23 L, SW24 ;, SW25 Bs, SW26 Shift(L), SW27 Z, SW28 X, SW29 C, SW3 W, SW30 V, SW31 B, SW32 N, SW33 M, SW34 ,, SW35 ., SW36 Shift(R), SW37 Fn, SW38 Ctrl(L), SW39 Win(L), SW4 E, SW40 Alt(L), SW41 Shift(C), SW42 Fn(C), SW43 Enter, SW44 ←, SW45 ↓, SW46 ↑, SW47 →, SW5 R, SW6 T, SW7 Y, SW8 U, SW9 I, U1 MOUDLE-SEEEDUINO-XIAO

Commit message: feat: change PCB size(vertical)
Parts:
- moved H1 1.70 mm to (85.0, 87.2)
- moved H3 1.70 mm to (339.0, 87.2)
- moved H2 1.30 mm to (85.0, 155.7)
- moved H4 1.30 mm to (339.0, 155.7)
Other:
- board size 260 x 77.5 mm -> 260 x 76.5 mm
Changed lines of the file:
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@@
   )
   (footprint "kbd_Hole:m2_Screw_Hole" (layer "F.Cu")
-    (at 85 85.5)
+    (at 85 87.2)
     (descr "Mounting Hole 2.2mm, no annular, M2")
     (tags "mounting hole 2.2mm no annular m2")
@@
   )
   (footprint "kbd_Hole:m2_Screw_Hole" (layer "F.Cu")
-    (at 85 157)
+    (at 85 155.7)
     (descr "Mounting Hole 2.2mm, no annular, M2")
     (tags "mounting hole 2.2mm no annular m2")
@@
   )
   (footprint "kbd_Hole:m2_Screw_Hole" (layer "F.Cu")
-    (at 339 157)
+    (at 339 155.7)
     (descr "Mounting Hole 2.2mm, no annular, M2")
     (tags "mounting hole 2.2mm no annular m2")
@@
   )
   (footprint "kbd_Hole:m2_Screw_Hole" (layer "F.Cu")
-    (at 339 85.5)
+    (at 339 87.2)
     (descr "Mounting Hole 2.2mm, no annular, M2")
     (tags "mounting hole 2.2mm no annular m2")
@@
     )
   )
-  (gr_arc (start 340 82.5) (mid 341.414214 83.085786) (end 342 84.5) (layer "Edge.Cuts") (width 0.1))
-  (gr_arc (start 342 158) (mid 341.414214 159.414214) (end 340 160) (layer "Edge.Cuts") (width 0.1))
-  (gr_line (start 342 158) (end 342 84.5) (layer "Edge.Cuts") (width 0.1))
-  (gr_arc (start 82 84.5) (mid 82.585786 83.085786) (end 84 82.5) (layer "Edge.Cuts") (width 0.1))
-  (gr_line (start 82 84.5) (end 82 158) (layer "Edge.Cuts") (width 0.1))
-  (gr_line (start 84 160) (end 340 160) (layer "Edge.Cuts") (width 0.1))
-  (gr_line (start 340 82.5) (end 84 82.5) (layer "Edge.Cuts") (width 0.1))
-  (gr_arc (start 84 160) (mid 82.585786 159.414214) (end 82 158) (layer "Edge.Cuts") (width 0.1))
-  (gr_text "Water47 ver1.0 @PCB Designed by multifeb13" (at 340.8 153 90) (layer "B.SilkS")
+  (gr_arc (start 340 83.2) (mid 341.414214 83.785786) (end 342 85.2) (layer "Edge.Cuts") (width 0.1))
+  (gr_arc (start 342 157.7) (mid 341.414214 159.114214) (end 340 159.7) (layer "Edge.Cuts") (width 0.1))
+  (gr_line (start 342 157.7) (end 342 85.2) (layer "Edge.Cuts") (width 0.1))
+  (gr_arc (start 82 85.2) (mid 82.585786 83.785786) (end 84 83.2) (layer "Edge.Cuts") (width 0.1))
+  (gr_line (start 82 85.2) (end 82 157.7) (layer "Edge.Cuts") (width 0.1))
+  (gr_line (start 84 159.7) (end 340 159.7) (layer "Edge.Cuts") (width 0.1))
+  (gr_line (start 340 83.2) (end 84 83.2) (layer "Edge.Cuts") (width 0.1))
+  (gr_arc (start 84 159.7) (mid 82.585786 159.114214) (end 82 157.7) (layer "Edge.Cuts") (width 0.1))
+  (gr_text "Water47 ver1.0 @PCB Designed by multifeb13" (at 337.5 153 90) (layer "B.SilkS")
     (effects (font (size 1 1) (thickness 0.125)) (justify right mirror))
   )
   (dimension (type aligned) (layer "Cmts.User")
-    (pts (xy 339 82.5) (xy 339 160))
+    (pts (xy 339 83.2) (xy 339 159.7))
     (height -8.9)
-    (gr_text "77.5000 mm" (at 346.75 121.25 90) (layer "Cmts.User")
+    (gr_text "76.5000 mm" (at 346.75 121.45 90) (layer "Cmts.User")
       (effects (font (size 1 1) (thickness 0.15)))
     )

Commit message: feat: first wiring
Parts:
- SW1, SW10, SW11, SW12, SW13, SW15, SW16, SW17, SW18, SW19, SW2, SW20, SW21, SW22, SW23, SW24, SW27, SW28, SW29, SW3, SW30, SW31, SW32, SW33, SW34, SW35, SW37, SW4, SW44, SW45, SW46, SW47, SW5, SW6, SW7, SW8, SW9: footprint multifeb13_kbd_KiCad_lib:Kailh_Choc_V1_Hotswap_via_1u -> multifeb13_kbd_KiCad_lib:Kailh_Choc_V2_1u_wo_anker
- SW14, SW36, SW38, SW39, SW40, SW42: footprint multifeb13_kbd_KiCad_lib:Kailh_Choc_V1_Hotswap_via_1.25u -> multifeb13_kbd_KiCad_lib:Kailh_Choc_V2_1.25u_wo_anker
- SW25, SW26: footprint multifeb13_kbd_KiCad_lib:Kailh_Choc_V1_Hotswap_via_1.75u -> multifeb13_kbd_KiCad_lib:Kailh_Choc_V2_1.75u_wo_anker
- SW41, SW43: footprint multifeb13_kbd_KiCad_lib:Kailh_Choc_V1_Hotswap_via_2u -> multifeb13_kbd_KiCad_lib:Kailh_Choc_V2_2u_wo_anker
- moved D49 147.8 mm to (240.7, 102.4), turned to 180 degrees
- moved D52 130.4 mm to (278.6, 92.9), turned to 90 degrees
- moved D48 128.3 mm to (221.4, 94.9), turned to 90 degrees
- moved D53 83.9 mm to (330.1, 115.7), turned to 0 degrees
- moved D55 82.6 mm to (297.7, 86.0)
- moved D50 40.9 mm to (146.8, 122.0), turned to 90 degrees
- moved D13 8.01 mm to (334.4, 88.8), turned to 90 degrees
- moved U1 4.75 mm to (325.3, 92.2)
- moved D54 3.90 mm to (198.8, 136.2)
- moved D51 3.57 mm to (264.0, 100.5)
- moved D43 3.15 mm to (245.1, 155.9)
- moved D40 2.92 mm to (152.2, 155.9)
- moved D41 2.92 mm to (183.2, 155.9)
- moved D46 2.92 mm to (311.7, 155.9)
- moved D42 2.91 mm to (214.1, 155.9)
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Connections:
- U1 pad 10: PIN7 -> PIN6
- U1 pad 11: PIN6 -> PIN4
- U1 pad 2: PIN2 -> unconnected-(U1-Pad2)
- U1 pad 3: PIN3 -> PIN5
- U1 pad 4: PIN4 -> PIN3
- U1 pad 7: PIN5 -> PIN8
- U1 pad 8: unconnected-(U1-Pad8) -> PIN7
- U1 pad 9: PIN8 -> PIN2
Routing:
- net PIN5: track 177.3 -> 415.6 mm
- net PIN2: track 252.1 -> 101.6 mm
- net Net-(D55-Pad1): track 102.1 -> 197.3 mm
- net PIN3: track 164.9 -> 246.8 mm
- net PIN7: track 231.8 -> 307.0 mm
- net PIN1: track 162.9 -> 230.1 mm
- net Net-(D50-Pad1): track 318.7 -> 356.1 mm, vias 1 -> 0
- net PIN8: track 169.3 -> 152.8 mm, vias 2 -> 0
- net Net-(D53-Pad1): track 286.2 -> 299.6 mm
- net Net-(D52-Pad1): track 298.7 -> 288.2 mm
- net PIN6: track 116.3 -> 125.3 mm
- net Net-(D54-Pad1): track 40.9 -> 49.2 mm
- net Net-(D49-Pad1): track 313.1 -> 305.2 mm
- net Net-(D13-Pad2): track 2.98 -> 8.18 mm
- net Net-(D51-Pad1): track 360.2 -> 356.4 mm
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
Commit message: fix: wiring
- wiring for SW pin 1
- unconnected wire warning
Routing:
- net Net-(D53-Pad1): track 299.6 -> 342.3 mm
- net Net-(D50-Pad1): track 356.1 -> 392.2 mm
- net Net-(D52-Pad1): track 288.2 -> 318.2 mm
- net Net-(D49-Pad1): track 305.2 -> 332.1 mm
- net Net-(D51-Pad1): track 356.4 -> 381.6 mm
- net Net-(D48-Pad1): track 290.7 -> 313.1 mm
- net Net-(D55-Pad1): track 197.3 -> 217.6 mm
- net Net-(D54-Pad1): track 49.2 -> 59.6 mm
- net PIN6: track 125.3 -> 124.5 mm

Commit message: fix: clearance between footprint and wire
Routing:
- net Net-(D53-Pad1): track 342.3 -> 335.4 mm
- net Net-(D50-Pad1): track 392.2 -> 390.2 mm
- net Net-(D55-Pad1): track 217.6 -> 216.7 mm
- net Net-(D49-Pad1): track 332.1 -> 332.7 mm
- net Net-(D51-Pad1): track 381.6 -> 381.1 mm

Commit message: feat: add silkscreen of MCU
Parts:
- U1: value MOUDLE-SEEEDUINO-XIAO -> Seeeduino XIAO
Changed lines of the file:
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@@
       (effects (font (size 0.889 0.889) (thickness 0.1016)))
     )
-    (fp_text value "MOUDLE-SEEEDUINO-XIAO" (at 0 2.75 90) (layer "F.SilkS") hide
-      (effects (font (size 0.6096 0.6096) (thickness 0.0762)))
+    (fp_text value "Seeeduino XIAO" (at 0 -3.275 90) (layer "B.SilkS")
+      (effects (font (size 0.6096 0.6096) (thickness 0.0762)) (justify mirror))
     )
     (fp_rect (start 3.350197 -6.785813) (end 5.128197 -4.118813) (layer "Dwgs.User") (width 0.12) (fill none))
