File: Water47/pcb/PCB_Layer/Water47_PCB_Layer.kicad_pcb (KiCad board)
At the start: 2 copper layers, 260 x 76.5 mm, 107 parts, among them SW1 Esc, SW10 O, SW11 P, SW12 -, SW13 Del, SW14 Cmd, SW15 A, SW16 S, SW17 D, SW18 F, SW19 G, SW2 Q, SW20 H, SW21 J, SW22 K, SW23 L, SW24 ;, SW25 Bs, SW26 Shift(L), SW27 Z, SW28 X, SW29 C, SW3 W, SW30 V, SW31 B, SW32 N, SW33 M, SW34 ,, SW35 ., SW36 Shift(R), SW37 Fn, SW38 Ctrl(L), SW39 Win(L), SW4 E, SW40 Alt(L), SW41 Shift(C), SW42 Fn(C), SW43 Enter, SW44 ←, SW45 ↓, SW46 ↑, SW47 →, SW5 R, SW6 T, SW7 Y, SW8 U, SW9 I, U1 MOUDLE-SEEEDUINO-XIAO

Commit message: feat: add mounting hole, set gerber path
Parts:
- added H5: MountingHole, kbd_Hole:m2_Spacer_Hole_hex, F.Cu at (339.0, 104.8)
- added H6: MountingHole, kbd_Hole:m2_Spacer_Hole_hex, F.Cu at (85.0, 104.8)
Changed lines of the file:
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@@
       (drillshape 0)
       (scaleselection 1)
-      (outputdirectory "../../gerber/PCB_Layer/")
+      (outputdirectory "../../gerber/02PCB_Layer/")
     )
   )
@@
       (net 22 "Net-(D24-Pad2)") (pinfunction "2") (pintype "passive"))
   )
+  (footprint "kbd_Hole:m2_Spacer_Hole_hex" (layer "F.Cu")
+    (at 85 104.8)
+    (descr "Mounting Hole 2.2mm, no annular, M2")
+    (tags "mounting hole 2.2mm no annular m2")
+    (property "Sheetfile" "Water47_PCB_Layer.kicad_sch")
+    (property "Sheetname" "")
+    (attr exclude_from_pos_files)
+    (fp_text reference "H6" (at 0 -3.2) (layer "F.Fab")
+      (effects (font (size 1 1) (thickness 0.15)))
+    )
+    (fp_text value "MountingHole" (at 0 3.2) (layer "F.Fab")
+      (effects (font (size 1 1) (thickness 0.15)))
+    )
+    (fp_line (start -1.2 -2.15) (end -2.4 0) (layer "Edge.Cuts") (width 0.1))
+    (fp_line (start -1.2 2.15) (end 1.2 2.15) (layer "Edge.Cuts") (width 0.1))
+    (fp_line (start 2.4 0) (end 1.2 -2.15) (layer "Edge.Cuts") (width 0.1))
+    (fp_line (start -2.4 0) (end -1.2 2.15) (layer "Edge.Cuts") (width 0.1))
+    (fp_line (start 1.2 2.15) (end 2.4 0) (layer "Edge.Cuts") (width 0.1))
+    (fp_line (start 1.2 -2.15) (end -1.2 -2.15) (layer "Edge.Cuts") (width 0.1))
+  )
   (footprint "multifeb13_kbd_KiCad_lib:Kailh_Choc_V2_1u_wo_anker" (layer "F.Cu")
     (at 188.11875 130.96875)
@@
     )
   )
-  (footprint "kbd_Parts:Diode_SMD" (layer "F.Cu")
+  (footprint "kbd_Hole:m2_Spacer_Hole_hex" (layer "F.Cu")
+    (at 339 104.8)
+    (descr "Mounting Hole 2.2mm, no annular, M2")
+    (tags "mounting hole 2.2mm no annular m2")
+    (property "Sheetfile" "Water47_PCB_Layer.kicad_sch")
+    (property "Sheetname" "")
+    (attr exclude_from_pos_files)
+    (fp_text reference "H5" (at 0 -3.2) (layer "F.Fab")
+      (effects (font (size 1 1) (thickness 0.15)))
+    )
+    (fp_text value "MountingHole" (at 0 3.2) (layer "F.Fab")
+      (effects (font (size 1 1) (thickness 0.15)))
+    )
+    (fp_line (start -1.2 2.15) (end 1.2 2.15) (layer "Edge.Cuts") (width 0.1))
+    (fp_line (start -1.2 -2.15) (end -2.4 0) (layer "Edge.Cuts") (width 0.1))
+    (fp_line (start 1.2 2.15) (end 2.4 0) (layer "Edge.Cuts") (width 0.1))
+    (fp_line (start 2.4 0) (end 1.2 -2.15) (layer "Edge.Cuts") (width 0.1))
+    (fp_line (start 1.2 -2.15) (end -1.2 -2.15) (layer "Edge.Cuts") (width 0.1))
+    (fp_line (start -2.4 0) (end -1.2 2.15) (layer "Edge.Cuts") (width 0.1))
+  )
+  (footprint "kbd_Parts:Diode_SMD" (layer "F.Cu")

Commit message: fix: mounting hole rotation
Parts:
- turned H5 to 90 degrees
- turned H6 to 90 degrees
Changed lines of the file:
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@@
   )
   (footprint "kbd_Hole:m2_Spacer_Hole_hex" (layer "F.Cu")
-    (at 85 104.8)
+    (at 85 104.8 90)
     (descr "Mounting Hole 2.2mm, no annular, M2")
     (tags "mounting hole 2.2mm no annular m2")
@@
     (property "Sheetname" "")
     (attr exclude_from_pos_files)
-    (fp_text reference "H6" (at 0 -3.2) (layer "F.Fab")
+    (fp_text reference "H6" (at 0 -3.2 90) (layer "F.Fab")
       (effects (font (size 1 1) (thickness 0.15)))
     )
-    (fp_text value "MountingHole" (at 0 3.2) (layer "F.Fab")
+    (fp_text value "MountingHole" (at 0 3.2 90) (layer "F.Fab")
       (effects (font (size 1 1) (thickness 0.15)))
     )
@@
   )
   (footprint "kbd_Hole:m2_Spacer_Hole_hex" (layer "F.Cu")
-    (at 339 104.8)
+    (at 339 104.8 90)
     (descr "Mounting Hole 2.2mm, no annular, M2")
     (tags "mounting hole 2.2mm no annular m2")
@@
     (property "Sheetname" "")
     (attr exclude_from_pos_files)
-    (fp_text reference "H5" (at 0 -3.2) (layer "F.Fab")
+    (fp_text reference "H5" (at 0 -3.2 90) (layer "F.Fab")
       (effects (font (size 1 1) (thickness 0.15)))
     )
-    (fp_text value "MountingHole" (at 0 3.2) (layer "F.Fab")
+    (fp_text value "MountingHole" (at 0 3.2 90) (layer "F.Fab")
       (effects (font (size 1 1) (thickness 0.15)))
     )
