File: Water47/pcb/Bottom/Water47_Bottom.kicad_sch (KiCad schematic)
At the start: 5 parts, among them U1 MOUDLE-SEEEDUINO-XIAO

Commit message: feat: ignore reference micon parts
Parts:
- U1: now left out of the parts list
Changed lines of the file:
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@@
   )
   (symbol (lib_id "MOUDLE-SEEEDUINO-XIAO:MOUDLE-SEEEDUINO-XIAO") (at 73.66 38.1 0) (unit 1)
-    (in_bom yes) (on_board yes) (fields_autoplaced)
+    (in_bom no) (on_board no) (fields_autoplaced)
     (property "Reference" "U1" (id 0) (at 74.93 20.32 0)
       (effects (font (size 1.27 1.27)) hide)
