File: Water47/pcb/Top/Water47_Top.kicad_sch (KiCad schematic)
At the start: 4 parts

Commit message: feat: change mounting spacer to hex
Parts:
- H1, H2, H3, H4: footprint kbd_Hole:m2_Screw_Hole -> kbd_Hole:m2_Spacer_Hole_hex
Changed lines of the file:
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@@
       (effects (font (size 1.27 1.27)) (justify left))
     )
-    (property "Footprint" "kbd_Hole:m2_Screw_Hole" (id 2) (at 22.86 68.58 0)
+    (property "Footprint" "kbd_Hole:m2_Spacer_Hole_hex" (id 2) (at 22.86 68.58 0)
       (effects (font (size 1.27 1.27)) hide)
     )
@@
       (effects (font (size 1.27 1.27)) (justify left))
     )
-    (property "Footprint" "kbd_Hole:m2_Screw_Hole" (id 2) (at 29.21 218.44 0)
+    (property "Footprint" "kbd_Hole:m2_Spacer_Hole_hex" (id 2) (at 29.21 218.44 0)
       (effects (font (size 1.27 1.27)) hide)
     )
@@
       (effects (font (size 1.27 1.27)) (justify left))
     )
-    (property "Footprint" "kbd_Hole:m2_Screw_Hole" (id 2) (at 212.09 217.17 0)
+    (property "Footprint" "kbd_Hole:m2_Spacer_Hole_hex" (id 2) (at 212.09 217.17 0)
       (effects (font (size 1.27 1.27)) hide)
     )
@@
       (effects (font (size 1.27 1.27)) (justify left))
     )
-    (property "Footprint" "kbd_Hole:m2_Screw_Hole" (id 2) (at 217.17 63.5 0)
+    (property "Footprint" "kbd_Hole:m2_Spacer_Hole_hex" (id 2) (at 217.17 63.5 0)
       (effects (font (size 1.27 1.27)) hide)
     )
@@
   (symbol_instances
     (path "/17fe6c74-7093-4ce3-b0e5-cd6b76f5155b"
-      (reference "H1") (unit 1) (value "MountingHole") (footprint "kbd_Hole:m2_Screw_Hole")
+      (reference "H1") (unit 1) (value "MountingHole") (footprint "kbd_Hole:m2_Spacer_Hole_hex")
     )
     (path "/bbde9b31-2ca1-42cc-a23f-bd08fc375c76"
-      (reference "H2") (unit 1) (value "MountingHole") (footprint "kbd_Hole:m2_Screw_Hole")
+      (reference "H2") (unit 1) (value "MountingHole") (footprint "kbd_Hole:m2_Spacer_Hole_hex")
     )
     (path "/f64ccafc-8d73-4e0d-a0a9-52c38f87dc6c"
-      (reference "H3") (unit 1) (value "MountingHole") (footprint "kbd_Hole:m2_Screw_Hole")
+      (reference "H3") (unit 1) (value "MountingHole") (footprint "kbd_Hole:m2_Spacer_Hole_hex")
     )
     (path "/caa5335b-ab47-478f-b510-96296c076797"
-      (reference "H4") (unit 1) (value "MountingHole") (footprint "kbd_Hole:m2_Screw_Hole")
+      (reference "H4") (unit 1) (value "MountingHole") (footprint "kbd_Hole:m2_Spacer_Hole_hex")
     )
   )
