File: Water47/pcb/Top/Water47_Top.kicad_pcb (KiCad board)
At the start: 2 copper layers, 260 x 76.5 mm, 51 parts, among them SW1 Esc, SW10 O, SW11 P, SW12 -, SW13 Del, SW14 Cmd, SW15 A, SW16 S, SW17 D, SW18 F, SW19 G, SW2 Q, SW20 H, SW21 J, SW22 K, SW23 L, SW24 ;, SW25 Bs, SW26 Shift(L), SW27 Z, SW28 X, SW29 C, SW3 W, SW30 V, SW31 B, SW32 N, SW33 M, SW34 ,, SW35 ., SW36 Shift(R), SW37 Fn, SW38 Ctrl(L), SW39 Win(L), SW4 E, SW40 Alt(L), SW41 Shift(C), SW42 Fn(C), SW43 Enter, SW44 ←, SW45 ↓, SW46 ↑, SW47 →, SW5 R, SW6 T, SW7 Y, SW8 U, SW9 I

Commit message: feat: change mounting spacer to hex
Parts:
- H1, H2, H3, H4: footprint kbd_Hole:m2_Screw_Hole -> kbd_Hole:m2_Spacer_Hole_hex
- turned H1 to 90 degrees
- turned H2 to 90 degrees
- turned H3 to 90 degrees
- turned H4 to 90 degrees
Changed lines of the file:
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@@
     (fp_line (start -9.525 9.525) (end 9.525 9.525) (layer "F.Fab") (width 0.15))
   )
-  (footprint "kbd_Hole:m2_Screw_Hole" (layer "F.Cu")
-    (at 85 87.2)
+  (footprint "kbd_Hole:m2_Spacer_Hole_hex" (layer "F.Cu")
+    (at 85 87.2 90)
     (descr "Mounting Hole 2.2mm, no annular, M2")
     (tags "mounting hole 2.2mm no annular m2")
-    (property "Sheetfile" "Water47_PCB_Layer.kicad_sch")
-    (property "Sheetname" "")
-    (autoplace_cost90 1)
+    (property "Sheetfile" "Water47_Top.kicad_sch")
+    (property "Sheetname" "")
     (attr exclude_from_pos_files)
-    (fp_text reference "H1" (at 0 -3.2) (layer "F.Fab")
-      (effects (font (size 1 1) (thickness 0.15)))
-    )
-    (fp_text value "MountingHole" (at 0 3.2) (layer "F.Fab") hide
-      (effects (font (size 1 1) (thickness 0.15)))
-    )
-    (fp_text user "${REFERENCE}" (at 0.3 0) (layer "F.Fab") hide
-      (effects (font (size 1 1) (thickness 0.15)))
-    )
-    (fp_circle (center 0 0) (end 2.2 0) (layer "Cmts.User") (width 0.15) (fill none))
-    (fp_circle (center 0 0) (end 2.45 0) (layer "F.CrtYd") (width 0.05) (fill none))
-    (pad "" np_thru_hole circle locked (at 0 0) (size 2.2 2.2) (drill 2.2) (layers *.Cu *.Mask))
+    (fp_text reference "H1" (at 0 -3.2 90) (layer "F.Fab")
+      (effects (font (size 1 1) (thickness 0.15)))
+    )
+    (fp_text value "MountingHole" (at 0 3.2 90) (layer "F.Fab")
+      (effects (font (size 1 1) (thickness 0.15)))
+    )
+    (fp_line (start 1.2 2.15) (end 2.4 0) (layer "Edge.Cuts") (width 0.1))
+    (fp_line (start -1.2 -2.15) (end -2.4 0) (layer "Edge.Cuts") (width 0.1))
+    (fp_line (start 2.4 0) (end 1.2 -2.15) (layer "Edge.Cuts") (width 0.1))
+    (fp_line (start 1.2 -2.15) (end -1.2 -2.15) (layer "Edge.Cuts") (width 0.1))
+    (fp_line (start -1.2 2.15) (end 1.2 2.15) (layer "Edge.Cuts") (width 0.1))
+    (fp_line (start -2.4 0) (end -1.2 2.15) (layer "Edge.Cuts") (width 0.1))
   )
   (footprint "kbd_SW_Hole:SW_Hole_1.25u" (layer "F.Cu")
@@
     (fp_line (start -11.90625 -9.525) (end -11.90625 9.525) (layer "F.Fab") (width 0.15))
   )
-  (footprint "kbd_Hole:m2_Screw_Hole" (layer "F.Cu")
-    (at 85 155.7)
+  (footprint "kbd_Hole:m2_Spacer_Hole_hex" (layer "F.Cu")
+    (at 85 155.7 90)
     (descr "Mounting Hole 2.2mm, no annular, M2")
     (tags "mounting hole 2.2mm no annular m2")
-    (property "Sheetfile" "Water47_PCB_Layer.kicad_sch")
+    (property "Sheetfile" "Water47_Top.kicad_sch")
     (property "Sheetname" "")
     (attr exclude_from_pos_files)
-    (fp_text reference "H2" (at 0 -3.2) (layer "F.Fab")
-      (effects (font (size 1 1) (thickness 0.15)))
-    )
-    (fp_text value "MountingHole" (at 0 3.2) (layer "F.Fab") hide
-      (effects (font (size 1 1) (thickness 0.15)))
-    )
-    (fp_text user "${REFERENCE}" (at 0.3 0) (layer "F.Fab") hide
-      (effects (font (size 1 1) (thickness 0.15)))
-    )
-    (fp_circle (center 0 0) (end 2.2 0) (layer "Cmts.User") (width 0.15) (fill none))
-    (fp_circle (center 0 0) (end 2.45 0) (layer "F.CrtYd") (width 0.05) (fill none))
-    (pad "" np_thru_hole circle locked (at 0 0) (size 2.2 2.2) (drill 2.2) (layers *.Cu *.Mask))
+    (fp_text reference "H2" (at 0 -3.2 90) (layer "F.Fab")
+      (effects (font (size 1 1) (thickness 0.15)))
+    )
+    (fp_text value "MountingHole" (at 0 3.2 90) (layer "F.Fab")
+      (effects (font (size 1 1) (thickness 0.15)))
+    )
+    (fp_line (start -1.2 2.15) (end 1.2 2.15) (layer "Edge.Cuts") (width 0.1))
+    (fp_line (start 1.2 2.15) (end 2.4 0) (layer "Edge.Cuts") (width 0.1))
+    (fp_line (start -2.4 0) (end -1.2 2.15) (layer "Edge.Cuts") (width 0.1))
+    (fp_line (start 1.2 -2.15) (end -1.2 -2.15) (layer "Edge.Cuts") (width 0.1))
+    (fp_line (start 2.4 0) (end 1.2 -2.15) (layer "Edge.Cuts") (width 0.1))
+    (fp_line (start -1.2 -2.15) (end -2.4 0) (layer "Edge.Cuts") (width 0.1))
   )
   (footprint "kbd_SW_Hole:SW_Hole_1u" (layer "F.Cu")
@@
     (fp_line (start 9.525 -9.525) (end -9.525 -9.525) (layer "F.Fab") (width 0.15))
   )
-  (footprint "kbd_Hole:m2_Screw_Hole" (layer "F.Cu")
-    (at 339 155.7)
+  (footprint "kbd_Hole:m2_Spacer_Hole_hex" (layer "F.Cu")
+    (at 339 155.7 90)
     (descr "Mounting Hole 2.2mm, no annular, M2")
     (tags "mounting hole 2.2mm no annular m2")
-    (property "Sheetfile" "Water47_PCB_Layer.kicad_sch")
+    (property "Sheetfile" "Water47_Top.kicad_sch")
     (property "Sheetname" "")
     (attr exclude_from_pos_files)
-    (fp_text reference "H4" (at 0 -3.2) (layer "F.Fab") hide
-      (effects (font (size 1 1) (thickness 0.15)))
-    )
-    (fp_text value "MountingHole" (at 0 3.2) (layer "F.Fab") hide
-      (effects (font (size 1 1) (thickness 0.15)))
-    )
-    (fp_text user "${REFERENCE}" (at 0.3 0) (layer "F.Fab") hide
-      (effects (font (size 1 1) (thickness 0.15)))
-    )
-    (fp_circle (center 0 0) (end 2.2 0) (layer "Cmts.User") (width 0.15) (fill none))
-    (fp_circle (center 0 0) (end 2.45 0) (layer "F.CrtYd") (width 0.05) (fill none))
-    (pad "" np_thru_hole circle locked (at 0 0) (size 2.2 2.2) (drill 2.2) (layers *.Cu *.Mask))
+    (fp_text reference "H4" (at 0 -3.2 90) (layer "F.Fab")
+      (effects (font (size 1 1) (thickness 0.15)))
+    )
+    (fp_text value "MountingHole" (at 0 3.2 90) (layer "F.Fab")
+      (effects (font (size 1 1) (thickness 0.15)))
+    )
+    (fp_line (start 2.4 0) (end 1.2 -2.15) (layer "Edge.Cuts") (width 0.1))
+    (fp_line (start -1.2 -2.15) (end -2.4 0) (layer "Edge.Cuts") (width 0.1))
+    (fp_line (start -2.4 0) (end -1.2 2.15) (layer "Edge.Cuts") (width 0.1))
+    (fp_line (start 1.2 -2.15) (end -1.2 -2.15) (layer "Edge.Cuts") (width 0.1))
+    (fp_line (start 1.2 2.15) (end 2.4 0) (layer "Edge.Cuts") (width 0.1))
+    (fp_line (start -1.2 2.15) (end 1.2 2.15) (layer "Edge.Cuts") (width 0.1))
   )
   (footprint "kbd_SW_Hole:SW_Hole_1u" (layer "F.Cu")
@@
     (fp_line (start 9.525 -9.525) (end -9.525 -9.525) (layer "F.Fab") (width 0.15))
   )
-  (footprint "kbd_Hole:m2_Screw_Hole" (layer "F.Cu")
-    (at 339 87.2)
+  (footprint "kbd_Hole:m2_Spacer_Hole_hex" (layer "F.Cu")
+    (at 339 87.2 90)
     (descr "Mounting Hole 2.2mm, no annular, M2")
     (tags "mounting hole 2.2mm no annular m2")
-    (property "Sheetfile" "Water47_PCB_Layer.kicad_sch")
+    (property "Sheetfile" "Water47_Top.kicad_sch")
     (property "Sheetname" "")
     (attr exclude_from_pos_files)
-    (fp_text reference "H3" (at 0 -3.2) (layer "F.Fab")
-      (effects (font (size 1 1) (thickness 0.15)))
-    )
-    (fp_text value "MountingHole" (at 0 3.2) (layer "F.Fab")
-      (effects (font (size 1 1) (thickness 0.15)))
-    )
-    (fp_text user "${REFERENCE}" (at 0.3 0) (layer "F.Fab") hide
-      (effects (font (size 1 1) (thickness 0.15)))
-    )
-    (fp_circle (center 0 0) (end 2.2 0) (layer "Cmts.User") (width 0.15) (fill none))
-    (fp_circle (center 0 0) (end 2.45 0) (layer "F.CrtYd") (width 0.05) (fill none))
-    (pad "" np_thru_hole circle locked (at 0 0) (size 2.2 2.2) (drill 2.2) (layers *.Cu *.Mask))
-  )
-  (footprint "kbd_SW_Hole:SW_Hole_1u" (layer "F.Cu")
+    (fp_text reference "H3" (at 0 -3.2 90) (layer "F.Fab")
+      (effects (font (size 1 1) (thickness 0.15)))
+    )
+    (fp_text value "MountingHole" (at 0 3.2 90) (layer "F.Fab")
+      (effects (font (size 1 1) (thickness 0.15)))
+    )
+    (fp_line (start -1.2 2.15) (end 1.2 2.15) (layer "Edge.Cuts") (width 0.1))
+    (fp_line (start -1.2 -2.15) (end -2.4 0) (layer "Edge.Cuts") (width 0.1))
+    (fp_line (start 1.2 -2.15) (end -1.2 -2.15) (layer "Edge.Cuts") (width 0.1))
+    (fp_line (start -2.4 0) (end -1.2 2.15) (layer "Edge.Cuts") (width 0.1))
+    (fp_line (start 1.2 2.15) (end 2.4 0) (layer "Edge.Cuts") (width 0.1))
+    (fp_line (start 2.4 0) (end 1.2 -2.15) (layer "Edge.Cuts") (width 0.1))
+  )
+  (footprint "kbd_SW_Hole:SW_Hole_1u" (layer "F.Cu")

Commit message: feat: change mounting hole
PCB : Hex
Others : Round
Parts:
- H1, H2, H3, H4: footprint kbd_Hole:m2_Spacer_Hole_hex -> kbd_Hole:m2_Screw_Hole
- turned H1 to 0 degrees
- turned H2 to 0 degrees
- turned H3 to 0 degrees
- turned H4 to 0 degrees
Other:
- board text added: "Water47 ver1.0 @Top Designed by multifeb13"
- board text removed: "Water47 ver1.0 @PCB Designed by multifeb13"
Changed lines of the file:
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@@
     (fp_line (start -9.525 9.525) (end 9.525 9.525) (layer "F.Fab") (width 0.15))
   )
-  (footprint "kbd_Hole:m2_Spacer_Hole_hex" (layer "F.Cu")
-    (at 85 87.2 90)
+  (footprint "kbd_Hole:m2_Screw_Hole" (layer "F.Cu")
+    (at 85 87.2)
     (descr "Mounting Hole 2.2mm, no annular, M2")
     (tags "mounting hole 2.2mm no annular m2")
@@
     (property "Sheetname" "")
     (attr exclude_from_pos_files)
-    (fp_text reference "H1" (at 0 -3.2 90) (layer "F.Fab")
-      (effects (font (size 1 1) (thickness 0.15)))
-    )
-    (fp_text value "MountingHole" (at 0 3.2 90) (layer "F.Fab")
-      (effects (font (size 1 1) (thickness 0.15)))
-    )
-    (fp_line (start 1.2 2.15) (end 2.4 0) (layer "Edge.Cuts") (width 0.1))
-    (fp_line (start -1.2 -2.15) (end -2.4 0) (layer "Edge.Cuts") (width 0.1))
-    (fp_line (start 2.4 0) (end 1.2 -2.15) (layer "Edge.Cuts") (width 0.1))
-    (fp_line (start 1.2 -2.15) (end -1.2 -2.15) (layer "Edge.Cuts") (width 0.1))
-    (fp_line (start -1.2 2.15) (end 1.2 2.15) (layer "Edge.Cuts") (width 0.1))
-    (fp_line (start -2.4 0) (end -1.2 2.15) (layer "Edge.Cuts") (width 0.1))
+    (fp_text reference "H1" (at 0 -3.2) (layer "F.Fab")
+      (effects (font (size 1 1) (thickness 0.15)))
+    )
+    (fp_text value "MountingHole" (at 0 3.2) (layer "F.Fab")
+      (effects (font (size 1 1) (thickness 0.15)))
+    )
+    (fp_text user "${REFERENCE}" (at 0.3 0) (layer "F.Fab")
+      (effects (font (size 1 1) (thickness 0.15)))
+    )
+    (fp_circle (center 0 0) (end 2.2 0) (layer "Cmts.User") (width 0.15) (fill none))
+    (fp_circle (center 0 0) (end 2.45 0) (layer "F.CrtYd") (width 0.05) (fill none))
+    (pad "" np_thru_hole circle locked (at 0 0) (size 2.2 2.2) (drill 2.2) (layers *.Cu *.Mask))
   )
   (footprint "kbd_SW_Hole:SW_Hole_1.25u" (layer "F.Cu")
@@
     (fp_line (start -11.90625 -9.525) (end -11.90625 9.525) (layer "F.Fab") (width 0.15))
   )
-  (footprint "kbd_Hole:m2_Spacer_Hole_hex" (layer "F.Cu")
-    (at 85 155.7 90)
+  (footprint "kbd_Hole:m2_Screw_Hole" (layer "F.Cu")
+    (at 85 155.7)
     (descr "Mounting Hole 2.2mm, no annular, M2")
     (tags "mounting hole 2.2mm no annular m2")
@@
     (property "Sheetname" "")
     (attr exclude_from_pos_files)
-    (fp_text reference "H2" (at 0 -3.2 90) (layer "F.Fab")
-      (effects (font (size 1 1) (thickness 0.15)))
-    )
-    (fp_text value "MountingHole" (at 0 3.2 90) (layer "F.Fab")
-      (effects (font (size 1 1) (thickness 0.15)))
-    )
-    (fp_line (start -1.2 2.15) (end 1.2 2.15) (layer "Edge.Cuts") (width 0.1))
-    (fp_line (start 1.2 2.15) (end 2.4 0) (layer "Edge.Cuts") (width 0.1))
-    (fp_line (start -2.4 0) (end -1.2 2.15) (layer "Edge.Cuts") (width 0.1))
-    (fp_line (start 1.2 -2.15) (end -1.2 -2.15) (layer "Edge.Cuts") (width 0.1))
-    (fp_line (start 2.4 0) (end 1.2 -2.15) (layer "Edge.Cuts") (width 0.1))
-    (fp_line (start -1.2 -2.15) (end -2.4 0) (layer "Edge.Cuts") (width 0.1))
+    (fp_text reference "H2" (at 0 -3.2) (layer "F.Fab")
+      (effects (font (size 1 1) (thickness 0.15)))
+    )
+    (fp_text value "MountingHole" (at 0 3.2) (layer "F.Fab")
+      (effects (font (size 1 1) (thickness 0.15)))
+    )
+    (fp_text user "${REFERENCE}" (at 0.3 0) (layer "F.Fab")
+      (effects (font (size 1 1) (thickness 0.15)))
+    )
+    (fp_circle (center 0 0) (end 2.2 0) (layer "Cmts.User") (width 0.15) (fill none))
+    (fp_circle (center 0 0) (end 2.45 0) (layer "F.CrtYd") (width 0.05) (fill none))
+    (pad "" np_thru_hole circle locked (at 0 0) (size 2.2 2.2) (drill 2.2) (layers *.Cu *.Mask))
   )
   (footprint "kbd_SW_Hole:SW_Hole_1u" (layer "F.Cu")
@@
     (fp_line (start 9.525 -9.525) (end -9.525 -9.525) (layer "F.Fab") (width 0.15))
   )
-  (footprint "kbd_Hole:m2_Spacer_Hole_hex" (layer "F.Cu")
-    (at 339 155.7 90)
+  (footprint "kbd_Hole:m2_Screw_Hole" (layer "F.Cu")
+    (at 339 155.7)
     (descr "Mounting Hole 2.2mm, no annular, M2")
     (tags "mounting hole 2.2mm no annular m2")
@@
     (property "Sheetname" "")
     (attr exclude_from_pos_files)
-    (fp_text reference "H4" (at 0 -3.2 90) (layer "F.Fab")
-      (effects (font (size 1 1) (thickness 0.15)))
-    )
-    (fp_text value "MountingHole" (at 0 3.2 90) (layer "F.Fab")
-      (effects (font (size 1 1) (thickness 0.15)))
-    )
-    (fp_line (start 2.4 0) (end 1.2 -2.15) (layer "Edge.Cuts") (width 0.1))
-    (fp_line (start -1.2 -2.15) (end -2.4 0) (layer "Edge.Cuts") (width 0.1))
-    (fp_line (start -2.4 0) (end -1.2 2.15) (layer "Edge.Cuts") (width 0.1))
-    (fp_line (start 1.2 -2.15) (end -1.2 -2.15) (layer "Edge.Cuts") (width 0.1))
-    (fp_line (start 1.2 2.15) (end 2.4 0) (layer "Edge.Cuts") (width 0.1))
-    (fp_line (start -1.2 2.15) (end 1.2 2.15) (layer "Edge.Cuts") (width 0.1))
+    (fp_text reference "H4" (at 0 -3.2) (layer "F.Fab")
+      (effects (font (size 1 1) (thickness 0.15)))
+    )
+    (fp_text value "MountingHole" (at 0 3.2) (layer "F.Fab")
+      (effects (font (size 1 1) (thickness 0.15)))
+    )
+    (fp_text user "${REFERENCE}" (at 0.3 0) (layer "F.Fab")
+      (effects (font (size 1 1) (thickness 0.15)))
+    )
+    (fp_circle (center 0 0) (end 2.2 0) (layer "Cmts.User") (width 0.15) (fill none))
+    (fp_circle (center 0 0) (end 2.45 0) (layer "F.CrtYd") (width 0.05) (fill none))
+    (pad "" np_thru_hole circle locked (at 0 0) (size 2.2 2.2) (drill 2.2) (layers *.Cu *.Mask))
   )
   (footprint "kbd_SW_Hole:SW_Hole_1u" (layer "F.Cu")
@@
     (fp_line (start 9.525 -9.525) (end -9.525 -9.525) (layer "F.Fab") (width 0.15))
   )
-  (footprint "kbd_Hole:m2_Spacer_Hole_hex" (layer "F.Cu")
-    (at 339 87.2 90)
+  (footprint "kbd_Hole:m2_Screw_Hole" (layer "F.Cu")
+    (at 339 87.2)
     (descr "Mounting Hole 2.2mm, no annular, M2")
     (tags "mounting hole 2.2mm no annular m2")
@@
     (property "Sheetname" "")
     (attr exclude_from_pos_files)
-    (fp_text reference "H3" (at 0 -3.2 90) (layer "F.Fab")
-      (effects (font (size 1 1) (thickness 0.15)))
-    )
-    (fp_text value "MountingHole" (at 0 3.2 90) (layer "F.Fab")
-      (effects (font (size 1 1) (thickness 0.15)))
-    )
-    (fp_line (start -1.2 2.15) (end 1.2 2.15) (layer "Edge.Cuts") (width 0.1))
-    (fp_line (start -1.2 -2.15) (end -2.4 0) (layer "Edge.Cuts") (width 0.1))
-    (fp_line (start 1.2 -2.15) (end -1.2 -2.15) (layer "Edge.Cuts") (width 0.1))
-    (fp_line (start -2.4 0) (end -1.2 2.15) (layer "Edge.Cuts") (width 0.1))
-    (fp_line (start 1.2 2.15) (end 2.4 0) (layer "Edge.Cuts") (width 0.1))
-    (fp_line (start 2.4 0) (end 1.2 -2.15) (layer "Edge.Cuts") (width 0.1))
+    (fp_text reference "H3" (at 0 -3.2) (layer "F.Fab")
+      (effects (font (size 1 1) (thickness 0.15)))
+    )
+    (fp_text value "MountingHole" (at 0 3.2) (layer "F.Fab")
+      (effects (font (size 1 1) (thickness 0.15)))
+    )
+    (fp_text user "${REFERENCE}" (at 0.3 0) (layer "F.Fab")
+      (effects (font (size 1 1) (thickness 0.15)))
+    )
+    (fp_circle (center 0 0) (end 2.2 0) (layer "Cmts.User") (width 0.15) (fill none))
+    (fp_circle (center 0 0) (end 2.45 0) (layer "F.CrtYd") (width 0.05) (fill none))
+    (pad "" np_thru_hole circle locked (at 0 0) (size 2.2 2.2) (drill 2.2) (layers *.Cu *.Mask))
   )
   (footprint "kbd_SW_Hole:SW_Hole_1u" (layer "F.Cu")
@@
   (gr_line (start 340 83.2) (end 84 83.2) (layer "Edge.Cuts") (width 0.1))
   (gr_arc (start 84 159.7) (mid 82.585786 159.114214) (end 82 157.7) (layer "Edge.Cuts") (width 0.1))
-  (gr_text "Water47 ver1.0 @PCB Designed by multifeb13" (at 339 153 90) (layer "B.SilkS")
+  (gr_text "Water47 ver1.0 @Top Designed by multifeb13" (at 339 153 90) (layer "B.SilkS")
     (effects (font (size 1 1) (thickness 0.125)) (justify right mirror))
   )

Commit message: fix: footprint rotation
Parts:
- turned SW13 to 0 degrees
Changed lines of the file:
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@@
   )
   (footprint "kbd_SW_Hole:SW_Hole_1u" (layer "F.Cu")
-    (at 326.23125 92.86875 180)
+    (at 326.23125 92.86875)
     (property "Sheetfile" "Water47_PCB_Layer.kicad_sch")
     (property "Sheetname" "")
     (attr through_hole)
-    (fp_text reference "SW13" (at 7 8.1 180) (layer "F.SilkS") hide
+    (fp_text reference "SW13" (at 7 8.1) (layer "F.SilkS") hide
       (effects (font (size 1 1) (thickness 0.15)))
     )
-    (fp_text value "Del" (at -7.4 -8.1 180) (layer "F.Fab") hide
+    (fp_text value "Del" (at -7.4 -8.1) (layer "F.Fab") hide
       (effects (font (size 1 1) (thickness 0.15)))
     )

Commit message: feat: add mounting hole, set gerber path
Parts:
- added H5: MountingHole, kbd_Hole:m2_Screw_Hole, F.Cu at (85.0, 104.8)
- added H6: MountingHole, kbd_Hole:m2_Screw_Hole, F.Cu at (339.0, 104.8)
Changed lines of the file:
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@@
       (drillshape 0)
       (scaleselection 1)
-      (outputdirectory "../../gerber/PCB_Layer1/")
+      (outputdirectory "../../gerber/01Top/")
     )
   )
@@
     (fp_line (start 9.525 -9.525) (end -9.525 -9.525) (layer "F.Fab") (width 0.15))
     (fp_line (start 9.525 9.525) (end 9.525 -9.525) (layer "F.Fab") (width 0.15))
+  )
+  (footprint "kbd_Hole:m2_Screw_Hole" (layer "F.Cu")
+    (at 85 104.8)
+    (descr "Mounting Hole 2.2mm, no annular, M2")
+    (tags "mounting hole 2.2mm no annular m2")
+    (property "Sheetfile" "Water47_Top.kicad_sch")
+    (property "Sheetname" "")
+    (attr exclude_from_pos_files)
+    (fp_text reference "H5" (at 0 -3.2) (layer "F.Fab")
+      (effects (font (size 1 1) (thickness 0.15)))
+    )
+    (fp_text value "MountingHole" (at 0 3.2) (layer "F.Fab")
+      (effects (font (size 1 1) (thickness 0.15)))
+    )
+    (fp_text user "${REFERENCE}" (at 0.3 0) (layer "F.Fab")
+      (effects (font (size 1 1) (thickness 0.15)))
+    )
+    (fp_circle (center 0 0) (end 2.2 0) (layer "Cmts.User") (width 0.15) (fill none))
+    (fp_circle (center 0 0) (end 2.45 0) (layer "F.CrtYd") (width 0.05) (fill none))
+    (pad "" np_thru_hole circle locked (at 0 0) (size 2.2 2.2) (drill 2.2) (layers *.Cu *.Mask))
   )
   (footprint "kbd_SW_Hole:SW_Hole_1u" (layer "F.Cu")
@@
     (fp_line (start 9.525 -9.525) (end -9.525 -9.525) (layer "F.Fab") (width 0.15))
   )
-  (footprint "kbd_SW_Hole:SW_Hole_1u" (layer "F.Cu")
+  (footprint "kbd_Hole:m2_Screw_Hole" (layer "F.Cu")
+    (at 339 104.8)
+    (descr "Mounting Hole 2.2mm, no annular, M2")
+    (tags "mounting hole 2.2mm no annular m2")
+    (property "Sheetfile" "Water47_Top.kicad_sch")
+    (property "Sheetname" "")
+    (attr exclude_from_pos_files)
+    (fp_text reference "H6" (at 0 -3.2) (layer "F.Fab")
+      (effects (font (size 1 1) (thickness 0.15)))
+    )
+    (fp_text value "MountingHole" (at 0 3.2) (layer "F.Fab")
+      (effects (font (size 1 1) (thickness 0.15)))
+    )
+    (fp_text user "${REFERENCE}" (at 0.3 0) (layer "F.Fab")
+      (effects (font (size 1 1) (thickness 0.15)))
+    )
+    (fp_circle (center 0 0) (end 2.2 0) (layer "Cmts.User") (width 0.15) (fill none))
+    (fp_circle (center 0 0) (end 2.45 0) (layer "F.CrtYd") (width 0.05) (fill none))
+    (pad "" np_thru_hole circle locked (at 0 0) (size 2.2 2.2) (drill 2.2) (layers *.Cu *.Mask))
+  )
+  (footprint "kbd_SW_Hole:SW_Hole_1u" (layer "F.Cu")
