File: Practice6/pcb/Bottom/Practice6_Bottom.kicad_pcb (KiCad board)
At the start: 2 copper layers, 61.5 x 42.5 mm, 8 parts

Commit message: feat: remove silkscreen
Parts:
- removed G***: LOGO, Silk_Wizard_logos:silk_wizard_logo_40x40
Other:
- board text removed: "Hurricane6 ver1.0 @Bottom Designed by multifeb13"
