File: Practice6/pcb/PCB_Layer/Practice6_PCB_Layer.kicad_pcb (KiCad board)
At the start: 2 copper layers, 61.5 x 42.5 mm, 19 parts, among them J1 Conn_01x03, SW1 SW_1, SW2 SW_2, SW3 SW_3, SW4 SW_4, SW5 SW_5, SW6 SW_6, U1 ProMicro

Commit message: feat: remove silkscreen
Other:
- board text removed: "Hurricane6 ver1.0 @PCB Designed by multifeb13"
Changed lines of the file:
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@@
   (gr_line (start 214.475 85.8) (end 156.975 85.8) (layer "Edge.Cuts") (width 0.1))
   (gr_arc (start 156.975 128.299986) (mid 155.560784 127.714202) (end 154.975 126.299986) (layer "Edge.Cuts") (width 0.1))
-  (gr_text "Hurricane6 ver1.0 @PCB\nDesigned by multifeb13" (at 161 125.592893) (layer "B.SilkS")
-    (effects (font (size 1 1) (thickness 0.125)) (justify right mirror))
-  )
   (dimension (type aligned) (layer "Cmts.User")
     (pts (xy 216.475 126.299986) (xy 154.975 126.299986))
